Commit message: Fix wheel joint and torque control; working wheel rotation

File: src/balance_bot/urdf/balance_bot.urdf.xacro (robot description, xacro)
@@ -8,7 +8,5 @@
   <xacro:property name="wheel_thickness" value="0.025"/>
   <xacro:property name="motor_length" value="0.03"/>
-  <xacro:property name="shaft_length" value="0.02"/>
-  <xacro:property name="shaft_radius" value="0.008"/>
-  <xacro:property name="stick_radius" value="0.002"/> <!-- 4 mm diameter -->
+  <xacro:property name="stick_radius" value="0.002"/>
   <xacro:property name="stick_length" value="0.4"/>
   <xacro:property name="wheel_diameter" value="${wheel_radius * 2}"/>
@@ -24,4 +22,21 @@
       </material>
     </visual>
+    <!-- Motor visuals inside base_plate -->
+    <visual>
+      <!-- Left motor -->
+      <geometry>
+        <cylinder radius="0.015" length="${motor_length}"/>
+      </geometry>
+      <origin xyz="${plate_length/2} 0 ${-plate_thickness/2 - 0.005}" rpy="0 1.5708 0"/>
+      <material name="Gray"/>
+    </visual>
+    <visual>
+      <!-- Right motor -->
+      <geometry>
+        <cylinder radius="0.015" length="${motor_length}"/>
+      </geometry>
+      <origin xyz="${-plate_length/2} 0 ${-plate_thickness/2 - 0.005}" rpy="0 1.5708 0"/>
+      <material name="Gray"/>
+    </visual>
     <collision>
       <geometry>
@@ -35,21 +50,22 @@
     </inertial>
   </link>
-<gazebo reference="base_plate">
-  <sensor type="imu" name="imu_sensor">
-    <always_on>true</always_on>
-    <update_rate>100.0</update_rate>
-    <visualize>true</visualize>
-    <plugin name="imu_plugin" filename="libgazebo_ros_imu_sensor.so">
-      <robotNamespace>/balance_bot</robotNamespace>
-      <topicName>imu_data</topicName>
-      <frameName>base_plate</frameName>
-      <updateRateHZ>100.0</updateRateHZ>
-      <gaussianNoise>0.0001</gaussianNoise>
-      <xyzOffset>0 0 0.402</xyzOffset>
-      <rpyOffset>0 0 0</rpyOffset>
-    </plugin>
-  </sensor>
-</gazebo>
-  <!-- Middle plate -->
+  <!-- IMU Sensor -->
+  <gazebo reference="base_plate">
+    <sensor type="imu" name="imu_sensor">
+      <always_on>true</always_on>
+      <update_rate>100.0</update_rate>
+      <visualize>true</visualize>
+      <plugin name="imu_plugin" filename="libgazebo_ros_imu_sensor.so">
+        <robotNamespace>/balance_bot</robotNamespace>
+        <topicName>imu_data</topicName>
+        <frameName>base_plate</frameName>
+        <updateRateHZ>100.0</updateRateHZ>
+        <gaussianNoise>0.0001</gaussianNoise>
+        <xyzOffset>0 0 0.402</xyzOffset>
+        <rpyOffset>0 0 0</rpyOffset>
+      </plugin>
+    </sensor>
+  </gazebo>
+  <!-- Middle and Top Plates -->
   <link name="middle_plate">
     <visual>
@@ -57,7 +73,5 @@
         <box size="${plate_length} ${plate_width} ${plate_thickness}"/>
       </geometry>
-      <material name="Gray">
-        <color rgba="0.6 0.6 0.6 1"/>
-      </material>
+      <material name="Gray"/>
     </visual>
     <collision>
@@ -76,5 +90,4 @@
     <origin xyz="0 0 ${stick_length/2}" />
   </joint>
-  <!-- Top plate -->
   <link name="top_plate">
     <visual>
@@ -82,7 +95,5 @@
         <box size="${plate_length} ${plate_width} ${plate_thickness}"/>
       </geometry>
-      <material name="Gray">
-        <color rgba="0.6 0.6 0.6 1"/>
-      </material>
+      <material name="Gray"/>
     </visual>
     <collision>
@@ -101,5 +112,5 @@
     <origin xyz="0 0 ${stick_length}" />
   </joint>
-  <!-- Sticks -->
+  <!-- 4 Sticks -->
   <xacro:macro name="stick" params="name x y">
     <link name="${name}">
@@ -109,7 +120,5 @@
         </geometry>
         <origin rpy="0 0 0"/>
-        <material name="DarkGray">
-          <color rgba="0.3 0.3 0.3 1"/>
-        </material>
+        <material name="DarkGray"/>
       </visual>
       <collision>
@@ -133,82 +142,85 @@
   <xacro:stick name="stick_bl" x="${-plate_length/2 + stick_radius}" y="${plate_width/2 - stick_radius}"/>
   <xacro:stick name="stick_br" x="${-plate_length/2 + stick_radius}" y="${-plate_width/2 + stick_radius}"/>
-  <!-- Motors and wheels (no mount) -->
-  <xacro:macro name="motor_assembly" params="side x_pos shaft_dir">
-    <xacro:property name="shaft_offset" value="${shaft_dir * (motor_length/2 + shaft_length/2)}"/>
-    <xacro:property name="wheel_offset" value="${shaft_dir * (shaft_length/2 + wheel_thickness/2)}"/>
-    <link name="${side}_motor">
-      <visual>
-        <geometry>
-          <cylinder radius="0.015" length="${motor_length}"/>
-        </geometry>
-        <origin rpy="0 1.5708 0"/>
-      </visual>
-      <collision>
-        <geometry>
-          <cylinder radius="0.015" length="${motor_length}"/>
-        </geometry>
-        <origin rpy="0 1.5708 0"/>
-      </collision>
-      <inertial>
-        <mass value="0.2"/>
-        <inertia ixx="2.6e-5" iyy="2.6e-5" izz="2.3e-5" ixy="0" ixz="0" iyz="0"/>
-      </inertial>
-    </link>
-    <joint name="${side}_motor_joint" type="fixed">
-      <parent link="base_plate"/>
-      <child link="${side}_motor"/>
-      <origin xyz="${x_pos} 0 ${-plate_thickness/2 - 0.005}"/> <!-- previous mount height -->
-    </joint>
-    <link name="${side}_shaft">
-      <visual>
-        <geometry>
-          <cylinder radius="${shaft_radius}" length="${shaft_length}"/>
-        </geometry>
-        <origin rpy="0 1.5708 0"/>
-      </visual>
-      <collision>
-        <geometry>
-          <cylinder radius="${shaft_radius}" length="${shaft_length}"/>
-        </geometry>
-        <origin rpy="0 1.5708 0"/>
-      </collision>
-      <inertial>
-        <mass value="0.05"/>
-        <inertia ixx="2.5e-6" iyy="2.5e-6" izz="1.6e-6" ixy="0" ixz="0" iyz="0"/>
-      </inertial>
-    </link>
-    <joint name="${side}_shaft_joint" type="revolute">
-      <parent link="${side}_motor"/>
-      <child link="${side}_shaft"/>
-      <origin xyz="${shaft_offset} 0 0"/>
-      <axis xyz="1 0 0"/>
-      <limit effort="5" velocity="10"/>
-    </joint>
-    <link name="${side}_wheel">
-      <visual>
-        <geometry>
-          <cylinder radius="${wheel_radius}" length="${wheel_thickness}"/>
-        </geometry>
-        <origin rpy="0 1.5708 0"/>
-      </visual>
-      <collision>
-        <geometry>
-          <cylinder radius="${wheel_radius}" length="${wheel_thickness}"/>
-        </geometry>
-        <origin rpy="0 1.5708 0"/>
-      </collision>
-      <inertial>
-        <mass value="0.2"/>
-        <inertia ixx="6.3e-5" iyy="6.3e-5" izz="1.1e-4" ixy="0" ixz="0" iyz="0"/>
-      </inertial>
-    </link>
-    <joint name="${side}_wheel_joint" type="continuous">
-      <parent link="${side}_shaft"/>
-      <child link="${side}_wheel"/>
-      <origin xyz="${wheel_offset} 0 0"/>
-      <axis xyz="1 0 0"/>
-    </joint>
-  </xacro:macro>
-  <xacro:motor_assembly side="left" x_pos="${plate_length/2}" shaft_dir="1"/>
-  <xacro:motor_assembly side="right" x_pos="${-plate_length/2}" shaft_dir="-1"/>
+  <!-- Wheels directly attached to base_plate at motor ends -->
+  <link name="left_wheel">
+    <visual>
+      <geometry>
+        <cylinder radius="${wheel_radius}" length="${wheel_thickness}"/>
+      </geometry>
+      <origin rpy="0 1.5708 0"/>
+    </visual>
+    <collision>
+      <geometry>
+        <cylinder radius="${wheel_radius}" length="${wheel_thickness}"/>
+      </geometry>
+      <origin rpy="0 1.5708 0"/>
+    </collision>
+    <inertial>
+      <mass value="0.2"/>
+      <inertia ixx="6.3e-5" iyy="6.3e-5" izz="1.1e-4" ixy="0" ixz="0" iyz="0"/>
+    </inertial>
+<gazebo>
+  <static>false</static>
+</gazebo>
+  </link>
+  <joint name="left_wheel_joint" type="continuous">
+    <parent link="base_plate"/>
+    <child link="left_wheel"/>
+    <origin xyz="${plate_length/2 + motor_length/2 + wheel_thickness/2} 0 ${-plate_thickness/2 - 0.005}" rpy="0 0 0"/>
+    <axis xyz="1 0 0"/>
+    <dynamics damping="0.1"/>
+  </joint>
+  <link name="right_wheel">
+    <visual>
+      <geometry>
+        <cylinder radius="${wheel_radius}" length="${wheel_thickness}"/>
+      </geometry>
+      <origin rpy="0 1.5708 0"/>
+    </visual>
+    <collision>
+      <geometry>
+        <cylinder radius="${wheel_radius}" length="${wheel_thickness}"/>
+      </geometry>
+      <origin rpy="0 1.5708 0"/>
+    </collision>
+    <inertial>
+      <mass value="0.2"/>
+      <inertia ixx="6.3e-5" iyy="6.3e-5" izz="1.1e-4" ixy="0" ixz="0" iyz="0"/>
+    </inertial>
+<gazebo>
+  <static>false</static>
+</gazebo>
+  </link>
+  <joint name="right_wheel_joint" type="continuous">
+    <parent link="base_plate"/>
+    <child link="right_wheel"/>
+    <origin xyz="${-plate_length/2 - motor_length/2 - wheel_thickness/2} 0 ${-plate_thickness/2 - 0.005}" rpy="0 0 0"/>
+    <axis xyz="1 0 0"/>
+    <dynamics damping="0.1"/>
+  </joint>
+<!-- Transmission definitions -->
+<transmission name="left_wheel_transmission">
+  <type>transmission_interface/SimpleTransmission</type>
+  <joint name="left_wheel_joint">
+    <hardwareInterface>hardware_interface/EffortJointInterface</hardwareInterface>
+  </joint>
+  <actuator name="left_wheel_motor">
+    <hardwareInterface>hardware_interface/EffortJointInterface</hardwareInterface>
+    <mechanicalReduction>1</mechanicalReduction>
+  </actuator>
+</transmission>
+<transmission name="right_wheel_transmission">
+  <type>transmission_interface/SimpleTransmission</type>
+  <joint name="right_wheel_joint">
+    <hardwareInterface>hardware_interface/EffortJointInterface</hardwareInterface>
+  </joint>
+  <actuator name="right_wheel_motor">
+    <hardwareInterface>hardware_interface/EffortJointInterface</hardwareInterface>
+    <mechanicalReduction>1</mechanicalReduction>
+  </actuator>
+</transmission>
+  <!-- ros_control plugin (important!) -->
+  <gazebo>
+    <plugin name="gazebo_ros_control" filename="libgazebo_ros_control.so"/>
+  </gazebo>
 </robot>

Commit message: simple pid

File: src/balance_bot/urdf/balance_bot.urdf.xacro (robot description, xacro)
@@ -144,24 +144,28 @@
   <!-- Wheels directly attached to base_plate at motor ends -->
   <link name="left_wheel">
-    <visual>
-      <geometry>
-        <cylinder radius="${wheel_radius}" length="${wheel_thickness}"/>
-      </geometry>
-      <origin rpy="0 1.5708 0"/>
-    </visual>
-    <collision>
-      <geometry>
-        <cylinder radius="${wheel_radius}" length="${wheel_thickness}"/>
-      </geometry>
-      <origin rpy="0 1.5708 0"/>
-    </collision>
-    <inertial>
-      <mass value="0.2"/>
-      <inertia ixx="6.3e-5" iyy="6.3e-5" izz="1.1e-4" ixy="0" ixz="0" iyz="0"/>
-    </inertial>
-<gazebo>
-  <static>false</static>
-</gazebo>
-  </link>
+  <visual>
+    <geometry>
+      <cylinder radius="${wheel_radius}" length="${wheel_thickness}"/>
+    </geometry>
+    <origin rpy="0 1.5708 0"/>
+  </visual>
+  <collision>
+    <geometry>
+      <cylinder radius="${wheel_radius}" length="${wheel_thickness}"/>
+    </geometry>
+    <origin rpy="0 1.5708 0"/>
+  </collision>
+  <inertial>
+    <mass value="0.2"/>
+    <inertia ixx="6.3e-5" iyy="6.3e-5" izz="1.1e-4" ixy="0" ixz="0" iyz="0"/>
+  </inertial>
+  <gazebo>
+    <static>false</static>
+    <mu1>1.0</mu1>
+    <mu2>1.0</mu2>
+    <kp>100000</kp>
+    <kd>1</kd>
+  </gazebo>
+</link>
   <joint name="left_wheel_joint" type="continuous">
     <parent link="base_plate"/>
@@ -172,24 +176,28 @@
   </joint>
   <link name="right_wheel">
-    <visual>
-      <geometry>
-        <cylinder radius="${wheel_radius}" length="${wheel_thickness}"/>
-      </geometry>
-      <origin rpy="0 1.5708 0"/>
-    </visual>
-    <collision>
-      <geometry>
-        <cylinder radius="${wheel_radius}" length="${wheel_thickness}"/>
-      </geometry>
-      <origin rpy="0 1.5708 0"/>
-    </collision>
-    <inertial>
-      <mass value="0.2"/>
-      <inertia ixx="6.3e-5" iyy="6.3e-5" izz="1.1e-4" ixy="0" ixz="0" iyz="0"/>
-    </inertial>
-<gazebo>
-  <static>false</static>
-</gazebo>
-  </link>
+  <visual>
+    <geometry>
+      <cylinder radius="${wheel_radius}" length="${wheel_thickness}"/>
+    </geometry>
+    <origin rpy="0 1.5708 0"/>
+  </visual>
+  <collision>
+    <geometry>
+      <cylinder radius="${wheel_radius}" length="${wheel_thickness}"/>
+    </geometry>
+    <origin rpy="0 1.5708 0"/>
+  </collision>
+  <inertial>
+    <mass value="0.2"/>
+    <inertia ixx="6.3e-5" iyy="6.3e-5" izz="1.1e-4" ixy="0" ixz="0" iyz="0"/>
+  </inertial>
+  <gazebo>
+    <static>false</static>
+    <mu1>1.0</mu1>
+    <mu2>1.0</mu2>
+    <kp>100000</kp>
+    <kd>1</kd>
+  </gazebo>
+</link>
   <joint name="right_wheel_joint" type="continuous">
     <parent link="base_plate"/>
@@ -224,3 +232,6 @@
     <plugin name="gazebo_ros_control" filename="libgazebo_ros_control.so"/>
   </gazebo>
+<gazebo reference="base_plate">
+  <pose>0 0 ${wheel_radius} 0 0 0</pose>
+</gazebo>
 </robot>

Commit message: PID with position

File: src/balance_bot/urdf/balance_bot.urdf.xacro (robot description, xacro)
@@ -47,5 +47,6 @@
     <inertial>
       <mass value="0.5"/>
-      <inertia ixx="2.8e-4" iyy="2.0e-3" izz="2.3e-3" ixy="0" ixz="0" iyz="0"/>
+      <!-- Approximated box inertia for base plate -->
+      <inertia ixx="0.00016" iyy="0.0020" izz="0.0020" ixy="0" ixz="0" iyz="0"/>
     </inertial>
   </link>
@@ -81,6 +82,7 @@
     </collision>
     <inertial>
-      <mass value="0.5"/>
-      <inertia ixx="2.8e-4" iyy="2.0e-3" izz="2.3e-3" ixy="0" ixz="0" iyz="0"/>
+      <mass value="0.1"/>
+      <!-- lighter inertia for thin plexiglass -->
+      <inertia ixx="3.5e-5" iyy="3.5e-5" izz="6.0e-5" ixy="0" ixz="0" iyz="0"/>
     </inertial>
   </link>
@@ -103,6 +105,7 @@
     </collision>
     <inertial>
-      <mass value="0.5"/>
-      <inertia ixx="2.8e-4" iyy="2.0e-3" izz="2.3e-3" ixy="0" ixz="0" iyz="0"/>
+      <mass value="0.1"/>
+      <!-- lighter inertia for thin plexiglass -->
+      <inertia ixx="3.5e-5" iyy="3.5e-5" izz="6.0e-5" ixy="0" ixz="0" iyz="0"/>
     </inertial>
   </link>
@@ -128,6 +131,7 @@
       </collision>
       <inertial>
-        <mass value="0.1"/>
-        <inertia ixx="1.3e-3" iyy="1.3e-3" izz="2.0e-7" ixy="0" ixz="0" iyz="0"/>
+        <mass value="0.05"/>
+        <!-- stick inertia for a thin rod -->
+        <inertia ixx="5.0e-5" iyy="5.0e-5" izz="2.0e-6" ixy="0" ixz="0" iyz="0"/>
       </inertial>
     </link>
@@ -157,11 +161,12 @@
   </collision>
   <inertial>
-    <mass value="0.2"/>
-    <inertia ixx="6.3e-5" iyy="6.3e-5" izz="1.1e-4" ixy="0" ixz="0" iyz="0"/>
+    <mass value="0.15"/>
+    <!-- wheel inertia approx as cylinder -->
+    <inertia ixx="1.5e-4" iyy="1.5e-4" izz="3.0e-4" ixy="0" ixz="0" iyz="0"/>
   </inertial>
   <gazebo>
     <static>false</static>
-    <mu1>1.0</mu1>
-    <mu2>1.0</mu2>
+    <mu1>0.5</mu1>
+    <mu2>0.5</mu2>
     <kp>100000</kp>
     <kd>1</kd>
@@ -189,11 +194,12 @@
   </collision>
   <inertial>
-    <mass value="0.2"/>
-    <inertia ixx="6.3e-5" iyy="6.3e-5" izz="1.1e-4" ixy="0" ixz="0" iyz="0"/>
+    <mass value="0.15"/>
+    <!-- wheel inertia approx as cylinder -->
+    <inertia ixx="1.5e-4" iyy="1.5e-4" izz="3.0e-4" ixy="0" ixz="0" iyz="0"/>
   </inertial>
   <gazebo>
     <static>false</static>
-    <mu1>1.0</mu1>
-    <mu2>1.0</mu2>
+    <mu1>0.5</mu1>
+    <mu2>0.5</mu2>
     <kp>100000</kp>
     <kd>1</kd>
@@ -235,3 +241,11 @@
   <pose>0 0 ${wheel_radius} 0 0 0</pose>
 </gazebo>
+<gazebo>
+  <plugin name="odometry_plugin" filename="libgazebo_ros_p3d.so">
+    <update_rate>100.0</update_rate>
+    <bodyName>base_plate</bodyName> <!-- your robot's main base link -->
+    <topicName>odom</topicName>
+    <gaussianNoise>0.0</gaussianNoise>
+  </plugin>
+</gazebo>
 </robot>
