Commit message: new urdf but with collision

File: src/balance_bot/urdf/balance_bot.urdf.xacro (robot description, xacro)
@@ -8,6 +8,9 @@
   <xacro:property name="wheel_thickness" value="0.025"/>
   <xacro:property name="motor_length" value="0.03"/>
+  <xacro:property name="motor_radius" value="0.015"/>
+  <xacro:property name="shaft_length" value="0.01"/>
+  <xacro:property name="shaft_radius" value="0.005"/>
   <xacro:property name="stick_radius" value="0.002"/>
-  <xacro:property name="stick_length" value="0.2"/> <!-- about 20 cm -->
+  <xacro:property name="stick_length" value="0.2"/>
   <!-- === Base Plate === -->
   <link name="base_plate">
@@ -26,21 +29,156 @@
     <inertial>
       <mass value="1.0"/>
-      <inertia ixx="0.00054" iyy="0.0040" izz="0.0045"
-               ixy="0" ixz="0" iyz="0"/>
-    </inertial>
-<!-- Motors visuals -->
-  <visual>
-    <geometry>
-      <cylinder radius="0.015" length="${motor_length}"/>
-    </geometry>
-    <origin xyz="${plate_length/2} 0 ${-plate_thickness/2 - 0.005}" rpy="0 1.5708 0"/>
-  </visual>
-  <visual>
-    <geometry>
-      <cylinder radius="0.015" length="${motor_length}"/>
-    </geometry>
-    <origin xyz="${-plate_length/2} 0 ${-plate_thickness/2 - 0.005}" rpy="0 1.5708 0"/>
-  </visual>
-  </link>
+      <inertia ixx="0.00054" iyy="0.0040" izz="0.0045" ixy="0" ixz="0" iyz="0"/>
+    </inertial>
+  </link>
+<!-- === Motors === -->
+  <link name="left_motor">
+    <visual>
+      <geometry>
+        <cylinder radius="${motor_radius}" length="${motor_length}"/>
+      </geometry>
+      <origin rpy="0 1.5708 0"/>
+      <material name="DarkGray"/>
+    </visual>
+    <collision>
+      <geometry>
+        <cylinder radius="${motor_radius}" length="${motor_length}"/>
+      </geometry>
+      <origin rpy="0 1.5708 0"/>
+    </collision>
+    <inertial>
+      <mass value="0.05"/>
+      <inertia ixx="1e-5" iyy="1e-5" izz="1e-5" ixy="0" ixz="0" iyz="0"/>
+    </inertial>
+  </link>
+  <joint name="left_motor_joint" type="fixed">
+    <parent link="base_plate"/>
+    <child link="left_motor"/>
+    <origin xyz="${plate_length/2} 0 ${-plate_thickness/2 - motor_radius}"/>
+  </joint>
+  <link name="right_motor">
+    <visual>
+      <geometry>
+        <cylinder radius="${motor_radius}" length="${motor_length}"/>
+      </geometry>
+      <origin rpy="0 1.5708 0"/>
+      <material name="DarkGray"/>
+    </visual>
+    <collision>
+      <geometry>
+        <cylinder radius="${motor_radius}" length="${motor_length}"/>
+      </geometry>
+      <origin rpy="0 1.5708 0"/>
+    </collision>
+    <inertial>
+      <mass value="0.05"/>
+      <inertia ixx="1e-5" iyy="1e-5" izz="1e-5" ixy="0" ixz="0" iyz="0"/>
+    </inertial>
+  </link>
+  <joint name="right_motor_joint" type="fixed">
+    <parent link="base_plate"/>
+    <child link="right_motor"/>
+    <origin xyz="${-plate_length/2} 0 ${-plate_thickness/2 - motor_radius}"/>
+  </joint>
+  <!-- === Shafts === -->
+  <link name="left_shaft">
+    <visual>
+      <geometry>
+        <cylinder radius="${shaft_radius}" length="${shaft_length}"/>
+      </geometry>
+      <origin rpy="0 1.5708 0"/>
+      <material name="Silver"/>
+    </visual>
+    <collision>
+      <geometry>
+        <cylinder radius="${shaft_radius}" length="${shaft_length}"/>
+      </geometry>
+      <origin rpy="0 1.5708 0"/>
+    </collision>
+    <inertial>
+      <mass value="0.01"/>
+      <inertia ixx="1e-6" iyy="1e-6" izz="1e-6" ixy="0" ixz="0" iyz="0"/>
+    </inertial>
+  </link>
+  <joint name="left_shaft_joint" type="fixed">
+    <parent link="left_motor"/>
+    <child link="left_shaft"/>
+    <origin xyz="${motor_length/2 + shaft_length/2} 0 0"/>
+  </joint>
+  <link name="right_shaft">
+    <visual>
+      <geometry>
+        <cylinder radius="${shaft_radius}" length="${shaft_length}"/>
+      </geometry>
+      <origin rpy="0 1.5708 0"/>
+      <material name="Silver"/>
+    </visual>
+    <collision>
+      <geometry>
+        <cylinder radius="${shaft_radius}" length="${shaft_length}"/>
+      </geometry>
+      <origin rpy="0 1.5708 0"/>
+    </collision>
+    <inertial>
+      <mass value="0.01"/>
+      <inertia ixx="1e-6" iyy="1e-6" izz="1e-6" ixy="0" ixz="0" iyz="0"/>
+    </inertial>
+  </link>
+  <joint name="right_shaft_joint" type="fixed">
+    <parent link="right_motor"/>
+    <child link="right_shaft"/>
+    <origin xyz="${-motor_length/2 - shaft_length/2} 0 0"/>
+  </joint>
+  <!-- === Wheels === -->
+  <link name="left_wheel">
+    <visual>
+      <geometry>
+        <cylinder radius="${wheel_radius}" length="${wheel_thickness}"/>
+      </geometry>
+      <origin rpy="0 1.5708 0"/>
+    </visual>
+    <collision>
+      <geometry>
+        <cylinder radius="${wheel_radius}" length="${wheel_thickness}"/>
+      </geometry>
+      <origin rpy="0 1.5708 0"/>
+    </collision>
+    <inertial>
+      <mass value="0.05"/>
+      <inertia ixx="3.2e-6" iyy="3.2e-6" izz="6.4e-6" ixy="0" ixz="0" iyz="0"/>
+    </inertial>
+  </link>
+  <joint name="left_wheel_joint" type="continuous">
+    <parent link="left_shaft"/>
+    <child link="left_wheel"/>
+    <origin xyz="${shaft_length/2 + wheel_thickness/2} 0 0"/>
+    <axis xyz="1 0 0"/>
+    <dynamics damping="0.1"/>
+  </joint>
+  <link name="right_wheel">
+    <visual>
+      <geometry>
+        <cylinder radius="${wheel_radius}" length="${wheel_thickness}"/>
+      </geometry>
+      <origin rpy="0 1.5708 0"/>
+    </visual>
+    <collision>
+      <geometry>
+        <cylinder radius="${wheel_radius}" length="${wheel_thickness}"/>
+      </geometry>
+      <origin rpy="0 1.5708 0"/>
+    </collision>
+    <inertial>
+      <mass value="0.05"/>
+      <inertia ixx="3.2e-6" iyy="3.2e-6" izz="6.4e-6" ixy="0" ixz="0" iyz="0"/>
+    </inertial>
+  </link>
+  <joint name="right_wheel_joint" type="continuous">
+    <parent link="right_shaft"/>
+    <child link="right_wheel"/>
+    <origin xyz="${-shaft_length/2 - wheel_thickness/2} 0 0"/>
+    <axis xyz="1 0 0"/>
+    <dynamics damping="0.1"/>
+  </joint>
   <!-- === Middle Plate === -->
   <link name="middle_plate">
@@ -58,6 +196,5 @@
     <inertial>
       <mass value="0.1"/>
-      <inertia ixx="5.4e-5" iyy="0.00040" izz="0.00045"
-               ixy="0" ixz="0" iyz="0"/>
+      <inertia ixx="5.4e-5" iyy="0.00040" izz="0.00045" ixy="0" ixz="0" iyz="0"/>
     </inertial>
   </link>
@@ -65,5 +202,5 @@
     <parent link="base_plate"/>
     <child link="middle_plate"/>
-    <origin xyz="0 0 0.1"/> <!-- 10 cm above base -->
+    <origin xyz="0 0 0.1"/>
   </joint>
   <!-- === Top Plate === -->
@@ -82,6 +219,5 @@
     <inertial>
       <mass value="0.02"/>
-      <inertia ixx="1e-5" iyy="1e-5" izz="2e-5"
-               ixy="0" ixz="0" iyz="0"/>
+      <inertia ixx="1e-5" iyy="1e-5" izz="2e-5" ixy="0" ixz="0" iyz="0"/>
     </inertial>
   </link>
@@ -89,23 +225,6 @@
     <parent link="base_plate"/>
     <child link="top_plate"/>
-    <origin xyz="0 0 0.2"/> <!-- 20 cm above base -->
-  </joint>
-  <!-- === IMU === -->
-  <gazebo reference="middle_plate">
-    <sensor type="imu" name="imu_sensor">
-      <always_on>true</always_on>
-      <update_rate>200.0</update_rate>
-      <visualize>true</visualize>
-      <plugin name="imu_plugin" filename="libgazebo_ros_imu_sensor.so">
-        <robotNamespace>/balance_bot</robotNamespace>
-        <topicName>imu_data</topicName>
-        <frameName>middle_plate</frameName>
-        <updateRateHZ>200.0</updateRateHZ>
-        <gaussianNoise>0.0001</gaussianNoise>
-        <xyzOffset>0 0 0</xyzOffset>
-        <rpyOffset>0 0 0</rpyOffset>
-      </plugin>
-    </sensor>
-  </gazebo>
+    <origin xyz="0 0 0.2"/>
+  </joint>
   <!-- === 4 Sticks === -->
   <xacro:macro name="stick" params="name x y">
@@ -115,5 +234,4 @@
           <cylinder radius="${stick_radius}" length="${stick_length}"/>
         </geometry>
-        <origin rpy="0 0 0"/>
         <material name="DarkGray"/>
       </visual>
@@ -125,6 +243,5 @@
       <inertial>
         <mass value="0.03"/>
-        <inertia ixx="5e-5" iyy="5e-5" izz="2e-6"
-                 ixy="0" ixz="0" iyz="0"/>
+        <inertia ixx="5e-5" iyy="5e-5" izz="2e-6" ixy="0" ixz="0" iyz="0"/>
       </inertial>
     </link>
@@ -139,58 +256,5 @@
   <xacro:stick name="stick_bl" x="${-plate_length/2 + stick_radius}" y="${plate_width/2 - stick_radius}"/>
   <xacro:stick name="stick_br" x="${-plate_length/2 + stick_radius}" y="${-plate_width/2 + stick_radius}"/>
-  <!-- === Wheels === -->
-  <link name="left_wheel">
-    <visual>
-      <geometry>
-        <cylinder radius="${wheel_radius}" length="${wheel_thickness}"/>
-      </geometry>
-      <origin rpy="0 1.5708 0"/>
-    </visual>
-    <collision>
-      <geometry>
-        <cylinder radius="${wheel_radius}" length="${wheel_thickness}"/>
-      </geometry>
-      <origin rpy="0 1.5708 0"/>
-    </collision>
-    <inertial>
-      <mass value="0.05"/>
-      <inertia ixx="3.2e-6" iyy="3.2e-6" izz="6.4e-6"
-               ixy="0" ixz="0" iyz="0"/>
-    </inertial>
-  </link>
- <joint name="left_wheel_joint" type="continuous">
-    <parent link="base_plate"/>
-    <child link="left_wheel"/>
-    <origin xyz="${plate_length/2 + motor_length/2 + wheel_thickness/2} 0 -0.007" rpy="0 0 0"/>
-    <axis xyz="1 0 0"/>
-    <dynamics damping="0.1"/>
-  </joint>
-  <link name="right_wheel">
-    <visual>
-      <geometry>
-        <cylinder radius="${wheel_radius}" length="${wheel_thickness}"/>
-      </geometry>
-      <origin rpy="0 1.5708 0"/>
-    </visual>
-    <collision>
-      <geometry>
-        <cylinder radius="${wheel_radius}" length="${wheel_thickness}"/>
-      </geometry>
-      <origin rpy="0 1.5708 0"/>
-    </collision>
-    <inertial>
-      <mass value="0.05"/>
-      <inertia ixx="3.2e-6" iyy="3.2e-6" izz="6.4e-6"
-               ixy="0" ixz="0" iyz="0"/>
-    </inertial>
-  </link>
-  <joint name="right_wheel_joint" type="continuous">
-    <parent link="base_plate"/>
-    <child link="right_wheel"/>
-    <origin xyz="${-plate_length/2 - motor_length/2 - wheel_thickness/2} 0 -0.007" rpy="0 0 0"/>
-    <axis xyz="1 0 0"/>
-    <dynamics damping="0.1"/>
-  </joint>
-  <!-- === Transmission === -->
+  <!-- === Transmissions === -->
   <transmission name="left_wheel_transmission">
     <type>transmission_interface/SimpleTransmission</type>
@@ -225,3 +289,25 @@
     </plugin>
   </gazebo>
+<gazebo reference="imu_link">
+  <sensor type="imu" name="imu_sensor">
+    <always_on>true</always_on>
+    <update_rate>200.0</update_rate> <!-- Gazebo physics -->
+    <visualize>true</visualize>
+    <plugin name="imu_plugin" filename="libgazebo_ros_imu_sensor.so">
+      <robotNamespace>/balance_bot</robotNamespace>
+      <topicName>imu_data</topicName>
+      <frameName>imu_link</frameName>
+      <updateRateHZ>200.0</updateRateHZ> <!-- ROS plugin reads THIS -->
+      <gaussianNoise>0.0001</gaussianNoise>
+      <xyzOffset>0 0 0</xyzOffset>
+      <rpyOffset>0 0 0</rpyOffset>
+    </plugin>
+  </sensor>
+</gazebo>
+<link name="imu_link"/>
+<joint name="imu_joint" type="fixed">
+  <parent link="base_plate"/>
+  <child link="imu_link"/>
+  <origin xyz="0 0 0.1"/>
+</joint>
 </robot>

Commit message: final urdf

File: src/balance_bot/urdf/balance_bot.urdf.xacro (robot description, xacro)
@@ -1,4 +1,21 @@
 <?xml version="1.0"?>
 <robot name="balance_bot" xmlns:xacro="http://www.ros.org/wiki/xacro">
+<gazebo>
+    <physics type="ode">
+        <max_step_size>0.001</max_step_size>
+        <real_time_update_rate>1000</real_time_update_rate>
+        <solver_type>quick</solver_type>
+    </physics>
+</gazebo>
+  <!-- Material Definitions -->
+<material name="Gray">
+    <color rgba="0.7 0.7 0.7 1.0"/>
+</material>
+<material name="DarkGray">
+    <color rgba="0.3 0.3 0.3 1.0"/>
+</material>
+<material name="Silver">
+    <color rgba="0.8 0.8 0.8 1.0"/>
+</material>
   <!-- === Dimensions === -->
   <xacro:property name="plate_length" value="0.22"/>
@@ -149,11 +166,15 @@
     </inertial>
   </link>
-  <joint name="left_wheel_joint" type="continuous">
+<gazebo reference="left_wheel">
+    <mu1>2.0</mu1><mu2>2.0</mu2>
+    <kp>1e8</kp><kd>1000</kd>
+    <minDepth>0.001</minDepth>
+</gazebo>
+<joint name="left_wheel_joint" type="continuous">
     <parent link="left_shaft"/>
     <child link="left_wheel"/>
-    <origin xyz="${shaft_length/2 + wheel_thickness/2} 0 0"/>
-    <axis xyz="1 0 0"/>
-    <dynamics damping="0.1"/>
-  </joint>
+    <origin xyz="0.0175 0 0" rpy="0 0 0"/>  <!-- shaft_length/2 + wheel_thickness/2 -->
+    <axis xyz="0 1 0"/>  <!-- Should be Y axis for wheels -->
+</joint>
   <link name="right_wheel">
     <visual>
@@ -174,11 +195,15 @@
     </inertial>
   </link>
-  <joint name="right_wheel_joint" type="continuous">
+<gazebo reference="right_wheel">
+    <mu1>2.0</mu1><mu2>2.0</mu2>
+    <kp>1e8</kp><kd>1000</kd>
+    <minDepth>0.001</minDepth>
+</gazebo>
+<joint name="right_wheel_joint" type="continuous">
     <parent link="right_shaft"/>
     <child link="right_wheel"/>
-    <origin xyz="${-shaft_length/2 - wheel_thickness/2} 0 0"/>
-    <axis xyz="1 0 0"/>
-    <dynamics damping="0.1"/>
-  </joint>
+    <origin xyz="-0.0175 0 0" rpy="0 0 0"/>  <!-- shaft_length/2 + wheel_thickness/2 -->
+    <axis xyz="0 1 0"/>  <!-- Should be Y axis for wheels -->
+</joint>
   <!-- === Middle Plate === -->
   <link name="middle_plate">

Commit message: idk

File: src/balance_bot/urdf/balance_bot.urdf.xacro (robot description, xacro)
@@ -30,23 +30,23 @@
   <xacro:property name="stick_radius" value="0.002"/>
   <xacro:property name="stick_length" value="0.2"/>
-  <!-- === Base Plate === -->
-  <link name="base_plate">
-    <visual>
-      <geometry>
-        <box size="${plate_length} ${plate_width} ${plate_thickness}"/>
-      </geometry>
-      <origin xyz="0 0 0"/>
-      <material name="Gray"/>
-    </visual>
-    <collision>
-      <geometry>
-        <box size="${plate_length} ${plate_width} ${plate_thickness}"/>
-      </geometry>
-    </collision>
-    <inertial>
-      <mass value="1.0"/>
-      <inertia ixx="0.00054" iyy="0.0040" izz="0.0045" ixy="0" ixz="0" iyz="0"/>
-    </inertial>
-  </link>
+ <!-- === Base Plate === -->
+<link name="base_plate">
+  <visual>
+    <geometry>
+      <box size="${plate_length} ${plate_width} ${plate_thickness}"/>
+    </geometry>
+    <origin xyz="0 0 0"/>
+    <material name="Gray"/>
+  </visual>
+  <collision>
+    <geometry>
+      <box size="${plate_length} ${plate_width} ${plate_thickness}"/>
+    </geometry>
+  </collision>
+  <inertial>
+    <mass value="0.3"/>
+    <inertia ixx="0.00016" iyy="0.00121" izz="0.00171" ixy="0" ixz="0" iyz="0"/>
+  </inertial>
+</link>
 <!-- === Motors === -->
   <link name="left_motor">
@@ -147,62 +147,63 @@
     <origin xyz="${-motor_length/2 - shaft_length/2} 0 0"/>
   </joint>
-  <!-- === Wheels === -->
-  <link name="left_wheel">
-    <visual>
-      <geometry>
-        <cylinder radius="${wheel_radius}" length="${wheel_thickness}"/>
-      </geometry>
-      <origin rpy="0 1.5708 0"/>
-    </visual>
-    <collision>
-      <geometry>
-        <cylinder radius="${wheel_radius}" length="${wheel_thickness}"/>
-      </geometry>
-      <origin rpy="0 1.5708 0"/>
-    </collision>
-    <inertial>
-      <mass value="0.05"/>
-      <inertia ixx="3.2e-6" iyy="3.2e-6" izz="6.4e-6" ixy="0" ixz="0" iyz="0"/>
-    </inertial>
-  </link>
+<!-- === UPDATED WHEELS === -->
+<link name="left_wheel">
+  <visual>
+    <geometry>
+      <cylinder radius="${wheel_radius}" length="${wheel_thickness}"/>
+    </geometry>
+    <origin rpy="0 1.5708 0"/>
+  </visual>
+  <collision>
+    <geometry>
+      <cylinder radius="${wheel_radius}" length="${wheel_thickness}"/>
+    </geometry>
+    <origin rpy="0 1.5708 0"/>
+  </collision>
+  <inertial>
+    <mass value="0.05"/>
+    <inertia ixx="3.2e-6" iyy="3.2e-6" izz="6.4e-6" ixy="0" ixz="0" iyz="0"/>
+  </inertial>
+</link>
 <gazebo reference="left_wheel">
-    <mu1>2.0</mu1><mu2>2.0</mu2>
-    <kp>1e8</kp><kd>1000</kd>
-    <minDepth>0.001</minDepth>
+  <mu1>2.0</mu1><mu2>2.0</mu2>
+  <kp>1e6</kp><kd>1000</kd> <!-- Reduce for stability -->
+  <minDepth>0.001</minDepth>
 </gazebo>
 <joint name="left_wheel_joint" type="continuous">
-    <parent link="left_shaft"/>
-    <child link="left_wheel"/>
-    <origin xyz="0.0175 0 0" rpy="0 0 0"/>  <!-- shaft_length/2 + wheel_thickness/2 -->
-    <axis xyz="0 1 0"/>  <!-- Should be Y axis for wheels -->
+  <parent link="left_shaft"/>
+  <child link="left_wheel"/>
+  <!-- New offset: shaft_length/2 + wheel_thickness/2 -->
+  <origin xyz="${shaft_length/2 + wheel_thickness/2} 0 0"/>
+  <axis xyz="1 0 0"/>
 </joint>
-  <link name="right_wheel">
-    <visual>
-      <geometry>
-        <cylinder radius="${wheel_radius}" length="${wheel_thickness}"/>
-      </geometry>
-      <origin rpy="0 1.5708 0"/>
-    </visual>
-    <collision>
-      <geometry>
-        <cylinder radius="${wheel_radius}" length="${wheel_thickness}"/>
-      </geometry>
-      <origin rpy="0 1.5708 0"/>
-    </collision>
-    <inertial>
-      <mass value="0.05"/>
-      <inertia ixx="3.2e-6" iyy="3.2e-6" izz="6.4e-6" ixy="0" ixz="0" iyz="0"/>
-    </inertial>
-  </link>
+<link name="right_wheel">
+  <visual>
+    <geometry>
+      <cylinder radius="${wheel_radius}" length="${wheel_thickness}"/>
+    </geometry>
+    <origin rpy="0 1.5708 0"/>
+  </visual>
+  <collision>
+    <geometry>
+      <cylinder radius="${wheel_radius}" length="${wheel_thickness}"/>
+    </geometry>
+    <origin rpy="0 1.5708 0"/>
+  </collision>
+  <inertial>
+    <mass value="0.05"/>
+    <inertia ixx="3.2e-6" iyy="3.2e-6" izz="6.4e-6" ixy="0" ixz="0" iyz="0"/>
+  </inertial>
+</link>
 <gazebo reference="right_wheel">
-    <mu1>2.0</mu1><mu2>2.0</mu2>
-    <kp>1e8</kp><kd>1000</kd>
-    <minDepth>0.001</minDepth>
+  <mu1>2.0</mu1><mu2>2.0</mu2>
+  <kp>1e6</kp><kd>1000</kd>
+  <minDepth>0.001</minDepth>
 </gazebo>
 <joint name="right_wheel_joint" type="continuous">
-    <parent link="right_shaft"/>
-    <child link="right_wheel"/>
-    <origin xyz="-0.0175 0 0" rpy="0 0 0"/>  <!-- shaft_length/2 + wheel_thickness/2 -->
-    <axis xyz="0 1 0"/>  <!-- Should be Y axis for wheels -->
+  <parent link="right_shaft"/>
+  <child link="right_wheel"/>
+  <origin xyz="${-shaft_length/2 - wheel_thickness/2} 0 0"/>
+  <axis xyz="1 0 0"/>
 </joint>
   <!-- === Middle Plate === -->

Commit message: new IMU but still now working right

File: src/balance_bot/urdf/balance_bot.urdf.xacro (robot description, xacro)
@@ -1,22 +1,5 @@
 <?xml version="1.0"?>
 <robot name="balance_bot" xmlns:xacro="http://www.ros.org/wiki/xacro">
-<gazebo>
-    <physics type="ode">
-        <max_step_size>0.001</max_step_size>
-        <real_time_update_rate>1000</real_time_update_rate>
-        <solver_type>quick</solver_type>
-    </physics>
-</gazebo>
-  <!-- Material Definitions -->
-<material name="Gray">
-    <color rgba="0.7 0.7 0.7 1.0"/>
-</material>
-<material name="DarkGray">
-    <color rgba="0.3 0.3 0.3 1.0"/>
-</material>
-<material name="Silver">
-    <color rgba="0.8 0.8 0.8 1.0"/>
-</material>
-  <!-- === Dimensions === -->
+<!-- === Dimensions === -->
   <xacro:property name="plate_length" value="0.22"/>
   <xacro:property name="plate_width" value="0.08"/>
@@ -128,5 +111,5 @@
         <cylinder radius="${shaft_radius}" length="${shaft_length}"/>
       </geometry>
-      <origin rpy="0 1.5708 0"/>
+      <origin xyz="0 0 0" rpy="0 1.5708 0"/>
       <material name="Silver"/>
     </visual>
@@ -135,5 +118,5 @@
         <cylinder radius="${shaft_radius}" length="${shaft_length}"/>
       </geometry>
-      <origin rpy="0 1.5708 0"/>
+      <origin  xyz="0 0 0" rpy="0 1.5708 0"/>
     </collision>
     <inertial>
@@ -148,4 +131,5 @@
   </joint>
 <!-- === UPDATED WHEELS === -->
+<!-- LEFT WHEEL LINK -->
 <link name="left_wheel">
   <visual>
@@ -153,5 +137,6 @@
       <cylinder radius="${wheel_radius}" length="${wheel_thickness}"/>
     </geometry>
-    <origin rpy="0 1.5708 0"/>
+    <origin xyz="0 0 0" rpy="0 1.5708 0"/> <!-- Centered geometry -->
+    <material name="DarkGray"/>
   </visual>
   <collision>
@@ -159,5 +144,5 @@
       <cylinder radius="${wheel_radius}" length="${wheel_thickness}"/>
     </geometry>
-    <origin rpy="0 1.5708 0"/>
+    <origin xyz="0 0 0" rpy="0 1.5708 0"/> <!-- Same as visual -->
   </collision>
   <inertial>
@@ -166,16 +151,14 @@
   </inertial>
 </link>
-<gazebo reference="left_wheel">
-  <mu1>2.0</mu1><mu2>2.0</mu2>
-  <kp>1e6</kp><kd>1000</kd> <!-- Reduce for stability -->
-  <minDepth>0.001</minDepth>
-</gazebo>
+<!-- LEFT WHEEL JOINT -->
 <joint name="left_wheel_joint" type="continuous">
   <parent link="left_shaft"/>
   <child link="left_wheel"/>
-  <!-- New offset: shaft_length/2 + wheel_thickness/2 -->
-  <origin xyz="${shaft_length/2 + wheel_thickness/2} 0 0"/>
+  <!-- Position wheel center at shaft end -->
+  <origin xyz="${shaft_length/2 + wheel_thickness/2 + 0.001} 0 0" rpy="0 0 0"/>
   <axis xyz="1 0 0"/>
+<limit effort="1.0" velocity="100.0"/>
 </joint>
+<!-- RIGHT WHEEL LINK -->
 <link name="right_wheel">
   <visual>
@@ -183,5 +166,6 @@
       <cylinder radius="${wheel_radius}" length="${wheel_thickness}"/>
     </geometry>
-    <origin rpy="0 1.5708 0"/>
+    <origin xyz="0 0 0" rpy="0 1.5708 0"/> <!-- Centered geometry -->
+    <material name="DarkGray"/>
   </visual>
   <collision>
@@ -189,5 +173,5 @@
       <cylinder radius="${wheel_radius}" length="${wheel_thickness}"/>
     </geometry>
-    <origin rpy="0 1.5708 0"/>
+    <origin xyz="0 0 0" rpy="0 1.5708 0"/> <!-- Same as visual -->
   </collision>
   <inertial>
@@ -196,14 +180,12 @@
   </inertial>
 </link>
-<gazebo reference="right_wheel">
-  <mu1>2.0</mu1><mu2>2.0</mu2>
-  <kp>1e6</kp><kd>1000</kd>
-  <minDepth>0.001</minDepth>
-</gazebo>
+<!-- RIGHT WHEEL JOINT -->
 <joint name="right_wheel_joint" type="continuous">
   <parent link="right_shaft"/>
   <child link="right_wheel"/>
-  <origin xyz="${-shaft_length/2 - wheel_thickness/2} 0 0"/>
+  <!-- Position wheel center at shaft end (negative direction) -->
+  <origin xyz="${-(shaft_length/2 + wheel_thickness/2 + 0.001)} 0 0" rpy="0 0 0"/>
   <axis xyz="1 0 0"/>
+<limit effort="1.0" velocity="100.0"/>
 </joint>
   <!-- === Middle Plate === -->
